Commit message: remove the inertia of base_link
to suppress the warning "The root link base_link has an inertia specified in the URDF, but KDL does not support a root link with an inertia.  As a workaround, you can add an extra dummy link to your URDF."

File: ar3_description/urdf/ar3.urdf.xacro (robot description, xacro)
@@ -6,9 +6,9 @@
 <robot name="ar3">
   <link name="base_link">
-    <inertial>
+    <!--<inertial>
       <origin rpy="0 0 0" xyz="-4.6941E-06 0.054174 0.038824"/>
       <mass value="0.7102"/>
       <inertia ixx="0.0039943" ixy="3.697E-07" ixz="-5.7364E-08" iyy="0.0014946" iyz="-0.00036051" izz="0.0042554"/>
-    </inertial>
+    </inertial>-->
     <visual>
       <origin rpy="0 0 0" xyz="0 0 0"/>

Commit message: add post-processing pipeline chain

File: ar3_description/urdf/ar3.urdf.xacro (robot description, xacro)
@@ -54,5 +54,5 @@
     <child link="link_1"/>
     <axis xyz="0 0 1"/>
-    <limit lower="-2.96706" upper="2.96706" effort="0" velocity="0"/>
+    <limit lower="${-170.0 / 180.0 * pi}" upper="${170.0 / 180.0 * pi}" effort="0" velocity="0"/>
   </joint>
   <link name="link_2">
@@ -83,5 +83,5 @@
     <child link="link_2"/>
     <axis xyz="0 0 -1"/>
-    <limit lower="${-39.6 / 180.0 * pi}" upper="${pi / 2.0}" effort="0" velocity="0"/>
+    <limit lower="${-39.6 / 180.0 * pi}" upper="${90.0 / 180.0 * pi}" effort="0" velocity="0"/>
   </joint>
   <link name="link_3">
@@ -112,5 +112,5 @@
     <child link="link_3"/>
     <axis xyz="0 0 -1"/>
-    <limit lower="0.0174533" upper="2.5080381" effort="0" velocity="0"/>
+    <limit lower="${-100.0 / 180.0 * pi}" upper="${80.0 / 180.0 * pi}" effort="0" velocity="0"/>
   </joint>
   <link name="link_4">
@@ -141,5 +141,5 @@
     <child link="link_4"/>
     <axis xyz="0 0 -1"/>
-    <limit lower="-2.8710666" upper="2.8710666" effort="0" velocity="0"/>
+    <limit lower="${-70.0 / 180.0 * pi}" upper="${-164.5 / 180.0 * pi}" effort="0" velocity="0"/>
   </joint>
   <link name="link_5">
@@ -170,5 +170,5 @@
     <child link="link_5"/>
     <axis xyz="1 0 0"/>
-    <limit lower="-1.81776042" upper="1.81776042" effort="0" velocity="0"/>
+    <limit lower="${-90.0 / 180.0 * pi}" upper="${95.0 / 180.0 * pi}" effort="0" velocity="0"/>
   </joint>
   <link name="link_6">
@@ -199,5 +199,5 @@
     <child link="link_6"/>
     <axis xyz="0 0 1"/>
-    <limit lower="-2.5848326" upper="2.5848326" effort="0" velocity="0"/>
+    <limit lower="${-148.0 / 180.0 * pi}" upper="${148.0 / 180.0 * pi}" effort="0" velocity="0"/>
   </joint>
 </robot>

Commit message: fix joint4's upper limit

File: ar3_description/urdf/ar3.urdf.xacro (robot description, xacro)
@@ -141,5 +141,5 @@
     <child link="link_4"/>
     <axis xyz="0 0 -1"/>
-    <limit lower="${-70.0 / 180.0 * pi}" upper="${-164.5 / 180.0 * pi}" effort="0" velocity="0"/>
+    <limit lower="${-70.0 / 180.0 * pi}" upper="${164.5 / 180.0 * pi}" effort="0" velocity="0"/>
   </joint>
   <link name="link_5">

Commit message: add end effect link to urdf

File: ar3_description/urdf/ar3.urdf.xacro (robot description, xacro)
@@ -201,3 +201,10 @@
     <limit lower="${-148.0 / 180.0 * pi}" upper="${148.0 / 180.0 * pi}" effort="0" velocity="0"/>
   </joint>
+  <!-- end-effector frame-->
+  <link name="link_7"/>
+  <joint name="joint_7" type="fixed">
+    <origin rpy="0 0 0" xyz="0 0 0"/>
+    <parent link="link_6"/>
+    <child link="link_7"/>
+  </joint>
 </robot>
